File: hardware/counter-pneumatic-v1/counter-pneumatic-v1-G368.kicad_pcb (KiCad board)
At the start: 2 copper layers, 71.1 x 132.1 mm, 43 parts, among them CON1 AVR-ISP-6, J1 Conn_01x06_Female, J2 Conn_01x02, J3 SD_Card, SW1 SW_Push, SW2 SW_Push, U1 MPX10DP, U2 MPX10DP, U3 MCP1700-3302E_SOT23, U4 NCP551SN33T1G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

Commit message: Update v1 PDF schematics and output files
Parts:
- removed U3: MCP1700-3302E_SOT23, Package_TO_SOT_SMD:SOT-23
- added C10: 0,1uF, Capacitor_SMD:C_0805_2012Metric_Pad1.15x1.40mm_HandSolder, F.Cu at (217.6, 54.4)
- added D2: MBR0530, Diode_SMD:D_SOD-123, F.Cu at (203.2, 146.4)
- added J4: JMP, Connector_PinHeader_2.54mm:PinHeader_1x02_P2.54mm_Vertical, F.Cu at (222.2, 83.8)
- added J5: Conn_01x06_Female, Connector_PinSocket_2.54mm:PinSocket_1x06_P2.54mm_Vertical, F.Cu at (234.9, 65.4)
- added Q1: Q_PNP_BEC, Package_TO_SOT_SMD:SOT-23_Handsoldering, F.Cu at (191.8, 50.8)
- added R12: 18K, Resistor_SMD:R_0805_2012Metric_Pad1.15x1.40mm_HandSolder, F.Cu at (189.9, 55.4)
- added R13: 0 NC, Resistor_SMD:R_0805_2012Metric_Pad1.15x1.40mm_HandSolder, F.Cu at (188.0, 50.3)
- added R14: 200K, Resistor_SMD:R_0805_2012Metric_Pad1.15x1.40mm_HandSolder, F.Cu at (219.3, 144.2)
- added R15: 600K, Resistor_SMD:R_0805_2012Metric_Pad1.15x1.40mm_HandSolder, F.Cu at (219.3, 148.1)
- added SW3: SW_Reed, Resistor_THT:R_Axial_DIN0411_L9.9mm_D3.6mm_P25.40mm_Horizontal, F.Cu at (254.6, 90.8)
- C1, C2, C3, C4, C5, C6, C7, C8, C9: footprint Capacitor_SMD:C_0805_2012Metric_Pad1.29x1.40mm_HandSolder -> Capacitor_SMD:C_0805_2012Metric_Pad1.15x1.40mm_HandSolder
- R1: value 100K -> 300K; footprint Resistor_SMD:R_0805_2012Metric_Pad1.29x1.40mm_HandSolder -> Resistor_SMD:R_0805_2012Metric_Pad1.15x1.40mm_HandSolder
- R10: value R -> 300; footprint Resistor_SMD:R_0805_2012Metric_Pad1.29x1.40mm_HandSolder -> Resistor_SMD:R_0805_2012Metric_Pad1.15x1.40mm_HandSolder
- R11, R2, R3, R4, R5, R6, R7, R8, R9: footprint Resistor_SMD:R_0805_2012Metric_Pad1.29x1.40mm_HandSolder -> Resistor_SMD:R_0805_2012Metric_Pad1.15x1.40mm_HandSolder
- Y2: value 32768 Hz -> 32768 Hz 12,5 pF
- moved D1 41.9 mm to (211.5, 80.0), turned to 270 degrees
- moved R10 37.4 mm to (215.3, 81.3)
- moved R4 16.0 mm to (217.6, 66.0), turned to 180 degrees
- moved R7 14.2 mm to (217.6, 63.5), turned to 180 degrees
- moved R5 12.0 mm to (221.6, 61.4), turned to 270 degrees
- moved R9 11.1 mm to (221.6, 57.5)
- moved R3 9.34 mm to (213.6, 52.1), turned to 180 degrees
- moved U5 8.64 mm to (215.8, 58.8)
- moved U2 7.89 mm to (231.6, 58.8)
- moved R8 7.77 mm to (213.6, 54.4), turned to 180 degrees
- moved R6 3.91 mm to (213.6, 63.5), turned to 0 degrees
- moved SW2 3.47 mm to (212.8, 73.0)
- moved U1 1.98 mm to (203.0, 52.8)
- moved C7 1.63 mm to (218.4, 75.8)
- moved J1 1.27 mm to (226.1, 73.7)
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Connections:
- net Net-(J1-Pad2) renamed /TXD
- net Net-(J1-Pad3) renamed /RXD
- J1 pad 5: Net-(J1-Pad5) -> (no net)
- J3 pad 10: Net-(J3-Pad10) -> (no net)
- J3 pad 11: Net-(J3-Pad11) -> (no net)
- J3 pad 8: Net-(J3-Pad8) -> (no net)
- J3 pad 9: Net-(J3-Pad9) -> (no net)
- U1 pad 3: +3V3 -> Net-(Q1-Pad3)
- U2 pad 3: +3V3 -> Net-(Q1-Pad3)
- U4 pad 4: Net-(U4-Pad4) -> (no net)
- U7 pad 1: Net-(U7-Pad1) -> /SENSOR_EN
- U7 pad 10: Net-(U7-Pad10) -> (no net)
- U7 pad 11: Net-(U7-Pad11) -> (no net)
- U7 pad 12: /PWRON -> Net-(D2-Pad2)
- U7 pad 13: Net-(U7-Pad13) -> /BT_STATE
- U7 pad 22: Net-(U7-Pad22) -> (no net)
- U7 pad 25: Net-(U7-Pad25) -> (no net)
- U7 pad 26: Net-(U7-Pad26) -> /BT_EN
- U7 pad 9: Net-(U7-Pad9) -> (no net)
- U8 pad 7: Net-(U8-Pad7) -> (no net)
Routing:
- net Net-(R14-Pad2): track 0.00 -> 62.3 mm, vias 0 -> 4
- net Net-(D1-Pad2): track 75.5 -> 15.9 mm
- net Net-(D2-Pad2): track 0.00 -> 57.2 mm, vias 0 -> 2
- net Net-(SW3-Pad2): track 0.00 -> 57.1 mm, vias 0 -> 1
- net /BT_STATE: track 0.00 -> 56.6 mm, vias 0 -> 3
- net /PWRON: track 90.9 -> 37.5 mm, vias 3 -> 0
- net /SENSOR_EN: track 0.00 -> 53.4 mm, vias 0 -> 2
- net Net-(Q1-Pad3): track 0.00 -> 52.7 mm
- net /BT_EN: track 0.00 -> 45.5 mm, vias 0 -> 2
- net /RXD: track 22.1 -> 44.7 mm
- net /PRESSURE0: track 48.1 -> 62.1 mm, vias 0 -> 2
- net +BATT: track 65.9 -> 54.7 mm
- net Net-(R4-Pad2): track 30.0 -> 19.0 mm
- net /PRESSURE1: track 40.7 -> 49.8 mm
- net Net-(R5-Pad2): track 13.1 -> 20.7 mm
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Other:
- board text added: "+3.3V"
- board text added: "BT Serial"
- board text added: "DTR"
- board text added: "Debug"
- board text added: "Debug PWR"
- board text added: "EN"
- board text added: "GND"
- board text added: "ISP"
- board text added: "Pneumatic bike counter v 1.0"
- board text added: "Power ON"
- board text added: "RXD"
- board text added: "Reset"
- board text added: "Start"
- board text added: "TXD"
