File: hardware/counter-pneumatic-v1/counter-pneumatic-v1.sch (KiCad schematic (older format))
At the start: 44 parts, among them CON1 AVR-ISP-6, J1 Conn_01x06_Female, J2 Conn_01x02, J3 SD_Card, SW1 SW_Push, SW2 SW_Push, U1 MPX10DP, U2 MPX10DP, U3 MCP1700-3302E_SOT23, U4 NCP551SN33T1G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

Commit message: Update schematics
Parts:
- removed U3: MCP1700-3302E_SOT23, Package_TO_SOT_SMD:SOT-23, symbol Regulator_Linear:MCP1700-3302E_SOT23
- added C10: 0,1uF, Capacitor_SMD:C_0805_2012Metric_Pad1.29x1.40mm_HandSolder, symbol Device:C_Small
- added D2: MBR0530, Diode_SMD:D_SOD-123, symbol Diode:MBR0530
- added J4: JMP, symbol Connector:Conn_01x02_Male
- added J5: Conn_01x06_Female, symbol Connector:Conn_01x06_Female
- added MK10, MK7, MK8, MK9: Mounting_Hole, MountingHole:MountingHole_3.2mm_M3, symbol Mechanical:Mounting_Hole
- added Q1: Q_PNP_BEC, symbol Device:Q_PNP_BEC
- added R12: 18K, Resistor_SMD:R_0805_2012Metric_Pad1.29x1.40mm_HandSolder, symbol Device:R
- added R13: 0 NC, symbol Device:R
- added R14: 200K, Resistor_SMD:R_0805_2012Metric_Pad1.29x1.40mm_HandSolder, symbol Device:R
- added R15: 600K, Resistor_SMD:R_0805_2012Metric_Pad1.29x1.40mm_HandSolder, symbol Device:R
- added SW3: SW_Reed, symbol Switch:SW_Reed
- R1: value 100K -> 300K
- R10: value R -> 300
- Y2: value 32768 Hz -> 32768 Hz 12,5 pF
Connections:
- net labels added: BT_EN, BT_STATE, RXD, SENSOR_EN, TXD
- wire segments 178 -> 216
- no-connect marks 17 -> 11
Other:
- note added: "CTS"
- note added: "DTR"
- note added: "EN"
- note added: "GND"
- note added: "PWR_DBG"
- note added: "RXD"
- note added: "STATE"
- note added: "Start Bluetooth"
- note added: "TXD"
- note added: "VCC"

Commit message: Update v1 PDF schematics and output files
Parts:
- added unit 3 of U5
- C1, C10, C2, C3, C4, C5, C6, C7, C8, C9: footprint Capacitor_SMD:C_0805_2012Metric_Pad1.29x1.40mm_HandSolder -> Capacitor_SMD:C_0805_2012Metric_Pad1.15x1.40mm_HandSolder
- J4: footprint (none) -> Connector_PinHeader_2.54mm:PinHeader_1x02_P2.54mm_Vertical
- J5: footprint (none) -> Connector_PinSocket_2.54mm:PinSocket_1x06_P2.54mm_Vertical
- Q1: footprint (none) -> Package_TO_SOT_SMD:SOT-23_Handsoldering
- R1, R10, R11, R12, R14, R2, R3, R4, R5, R6, R7, R8, R9: footprint Resistor_SMD:R_0805_2012Metric_Pad1.29x1.40mm_HandSolder -> Resistor_SMD:R_0805_2012Metric_Pad1.15x1.40mm_HandSolder
- R13: footprint (none) -> Resistor_SMD:R_0805_2012Metric_Pad1.15x1.40mm_HandSolder
- R15: value 600K -> 620K; footprint Resistor_SMD:R_0805_2012Metric_Pad1.29x1.40mm_HandSolder -> Resistor_SMD:R_0805_2012Metric_Pad1.15x1.40mm_HandSolder
- SW3: footprint (none) -> Resistor_THT:R_Axial_DIN0411_L9.9mm_D3.6mm_P25.40mm_Horizontal
Connections:
- wire segments 216 -> 214
Other:
- note added: "V1 Errata:\n1. R14 и R15 надо поменять местами (R14 должен быть 620К, R15 – 200К)\n"
